Commit message: Heterogenous Rover Platform Support

File: assets/robots/perseverance/m2020_lidar.urdf (robot description, URDF)
Before this commit: robot Perseverance, 86 links, 85 joints
Links:
- link Body_BogieLeft: geometry visual mesh filename=meshes/Left_Bogie.gltf scale=1 1 1
- link Body_BogieRight: geometry visual mesh filename=meshes/Right_Bogie.gltf scale=1 1 1
- link Body_Chassis: geometry visual mesh filename=../sensors/lidar_2d.obj; visual mesh filename=../sensors/lidar_3d.obj
- link Body_Differential: geometry visual mesh filename=meshes/CenterDifferential.gltf scale=1 1 1
- link Body_HGA_AZ: geometry visual mesh filename=meshes/HGA_AZ.gltf scale=1 1 1
- link Body_HGA_EL: geometry visual mesh filename=meshes/HGA_EL.gltf scale=1 1 1
- link Body_RSM_AZ: geometry visual mesh filename=meshes/RSM.gltf scale=1 1 1
- link Body_RSM_EL: geometry visual mesh filename=meshes/RSM_Head.gltf scale=1 1 1
- link Body_RockerLeft: geometry visual mesh filename=meshes/Left_Rocker.gltf scale=1 1 1
- link Body_RockerRight: geometry visual mesh filename=meshes/Right_Rocker.gltf scale=1 1 1
- link Body_SteerLeftFront: geometry visual mesh filename=meshes/Steer_LeftFront.gltf scale=1 1 1
- link Body_SteerLeftRear: geometry visual mesh filename=meshes/Steer_LeftRear.gltf scale=1 1 1
- link Body_SteerRightFront: geometry visual mesh filename=meshes/Steer_RightFront.gltf scale=1 1 1
- link Body_SteerRightRear: geometry visual mesh filename=meshes/Steer_RightRear.gltf scale=1 1 1
- link Body_WheelLeftFront: geometry visual mesh filename=meshes/Wheel_LeftFront.gltf scale=1 1 1
- link Body_WheelLeftMiddle: geometry visual mesh filename=meshes/Wheel_LeftMiddle.gltf scale=1 1 1
- link Body_WheelLeftRear: geometry visual mesh filename=meshes/Wheel_LeftRear.gltf scale=1 1 1
- link Body_WheelRightFront: geometry visual mesh filename=meshes/Wheel_RightFront.gltf scale=1 1 1
- link Body_WheelRightMiddle: geometry visual mesh filename=meshes/Wheel_RightMiddle.gltf scale=1 1 1
- link Body_WheelRightRear: geometry visual mesh filename=meshes/Wheel_RightRear.gltf scale=1 1 1
